Commit message: Update urdf so that joints are in correct starting locations and turn the correct direction

File: catkin_ws/src/dexter/urdf/robot.urdf (robot description, URDF)
Before this commit: robot dexter, 16 links, 15 joints
Joints:
- joint kp0093_1_kp0093_1_230_kp0028-01_armbodybottom_fixing: origin xyz=0.057 -0.037 0.0 rpy=0.0 0.673 1.571 -> xyz=0.057 -0.037 0.0 rpy=0.0 0.0 1.571
- joint kp0093_1_kp0093_1_237_kp0066-01_endarmhubbottom_fixing: origin xyz=0.0 -0.051 0.0 rpy=0.000 1.549 -3.142 -> xyz=0.0 -0.051 0.0 rpy=0.0 3.142 -3.142
- joint kp0093_1_kp0093_1_322_kp0079-01_diffa2codediskendstopfilled_fixing: axis 0 1 0 -> 0 -1 0; origin xyz=0.0 -0.024 0.0 rpy=0.0 -0.422 0.0 -> xyz=0.0 -0.024 0.0 rpy=0.0 0.0 0.0
- joint kp0093_1_kp0093_1_87_kp0086-01_outterfrontdifferentialgear_fixing: axis 0 1 0 -> 0 -1 0; origin xyz=0.021 -0.021 -0.021 rpy=-0.206 1.571 2.936 -> xyz=0.021 -0.021 -0.021 rpy=0.206 -1.571 2.936

Commit message: Add joint limits, rename joints to match documentation

File: catkin_ws/src/dexter/urdf/robot.urdf (robot description, URDF)
Before this commit: robot dexter, 16 links, 15 joints
Joints:
- removed joint kp0093_1_kp0093_1_183_kp0013-01_mainpivotv2_fixing
- removed joint kp0093_1_kp0093_1_230_kp0028-01_armbodybottom_fixing
- removed joint kp0093_1_kp0093_1_237_kp0066-01_endarmhubbottom_fixing
- removed joint kp0093_1_kp0093_1_322_kp0079-01_diffa2codediskendstopfilled_fixing
- removed joint kp0093_1_kp0093_1_87_kp0086-01_outterfrontdifferentialgear_fixing
- added joint J1: type revolute, parent kp0093_1_33_kp0021-01_motorendcappivot, child kp0093_1_183_kp0013-01_mainpivotv2, origin xyz=0.0 -0.008 0.0 rpy=0.0 0.0 0.0, axis 0 1 0, limit lower=-3.142 upper=3.142 effort=100 velocity=100
- added joint J2: type revolute, parent kp0093_1_183_kp0013-01_mainpivotv2, child kp0093_1_230_kp0028-01_armbodybottom, origin xyz=0.057 -0.037 0.0 rpy=0.0 0.0 1.571, axis 0 1 0, limit lower=-2.355 upper=2.355 effort=100 velocity=100
- added joint J3: type revolute, parent kp0093_1_48_kp0048-01_axisintersectionhalfsm_b, child kp0093_1_237_kp0066-01_endarmhubbottom, origin xyz=0.0 -0.051 0.0 rpy=0.0 3.142 -3.142, axis 0 1 0, limit lower=-2.355 upper=2.355 effort=100 velocity=100
- added joint J4: type revolute, parent kp0093_1_2_kp0070-01_endaxishubc, child kp0093_1_322_kp0079-01_diffa2codediskendstopfilled, origin xyz=0.0 -0.024 0.0 rpy=0.0 0.0 0.0, axis 0 -1 0, limit lower=-1.571 upper=1.571 effort=100 velocity=100
- added joint J5: type revolute, parent kp0093_1_12_kp0077-01_diffbodysmallb, child kp0093_1_87_kp0086-01_outterfrontdifferentialgear, origin xyz=0.021 -0.021 -0.021 rpy=0.206 -1.571 2.936, axis 0 -1 0, limit lower=-3.14 upper=3.14 effort=100 velocity=100

Commit message: Change Joint 1 values based on specific robot calibration (should be 360 degrees total

File: catkin_ws/src/dexter/urdf/robot.urdf (robot description, URDF)
Before this commit: robot dexter, 16 links, 15 joints
Joints:
- joint J1: limit lower=-3.142 upper=3.142 effort=100 velocity=100 -> lower=-1.571 upper=1.571 effort=100 velocity=100
